File: maveric-board/active_high_1v2_led.kicad_sch (KiCad schematic)
At the start: 4 parts, among them Q2 DMN2005K-7

Commit message: add uni2 socket footprint, check against drawing, fix npth, assign all footprints and part numbers
Parts:
- R18: footprint (none) -> Resistor_SMD:R_0603_1608Metric; JLCPCB Part # C25076 -> C22775
Changed lines of the file:
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@@
 			)
 		)
-		(property "Footprint" ""
+		(property "Footprint" "Resistor_SMD:R_0603_1608Metric"
 			(at 46.736 28.194 90)
 			(effects
@@
 			)
 		)
-		(property "Description" "Resistor, US symbol"
+		(property "Description" "0603WAF1000T5E"
 			(at 45.72 27.94 0)
 			(effects
@@
 			)
 		)
-		(property "JLCPCB Part #" "C25076"
+		(property "JLCPCB Part #" "C22775"
 			(at 45.72 27.94 0)
 			(effects
